File: board/akuhei.sch (KiCad schematic (older format))
At the start: 9 parts, among them J1 CLOCKPORT, J2 I2C, U2 PCA9564, U3 TLV70233DBV

Commit message: removing error
Connections:
- net A1: now also J1.12 (A2(30)); no longer J1.11 (A3(29))
- net A2: now also J1.11 (A3(29)); no longer J1.12 (A2(30))
Changed lines of the file:
@@
 CP_IOWR
-Entry Wire Line
-	3700 2300 3800 2400
 Entry Wire Line
 	3700 2400 3800 2500
@@
 Text GLabel 6150 2600 2    39   Input ~ 0
 CP_IOWR
-Text Label 1350 2300 0    39   ~ 0
+Text Label 3650 2300 0    39   ~ 0
 A1
 Text Label 3650 2700 0    39   ~ 0
@@
 $EndComp
 $Comp
-L +3.3V #PWR013
+L +3.3V #PWR07
 U 1 1 55CF94C4
 P 5250 1200
-F 0 "#PWR013" H 5250 1050 50  0001 C CNN
+F 0 "#PWR07" H 5250 1050 50  0001 C CNN
 F 1 "+3.3V" H 5250 1340 50  0000 C CNN
 F 2 "" H 5250 1200 60  0000 C CNN
@@
 $EndComp
 $Comp
-L GND #PWR014
+L GND #PWR08
 U 1 1 55CF94E4
 P 5250 3200
-F 0 "#PWR014" H 5250 2950 50  0001 C CNN
+F 0 "#PWR08" H 5250 2950 50  0001 C CNN
 F 1 "GND" H 5250 3050 50  0000 C CNN
 F 2 "" H 5250 3200 60  0000 C CNN
@@
 $EndComp
 $Comp
-L +5V #PWR015
+L +5V #PWR09
 U 1 1 55CFA1FC
 P 9100 2400
-F 0 "#PWR015" H 9100 2250 50  0001 C CNN
+F 0 "#PWR09" H 9100 2250 50  0001 C CNN
 F 1 "+5V" H 9100 2540 50  0000 C CNN
 F 2 "" H 9100 2400 60  0000 C CNN
@@
 $EndComp
 $Comp
-L +3.3V #PWR016
+L +3.3V #PWR010
 U 1 1 55CFA325
 P 10400 2400
-F 0 "#PWR016" H 10400 2250 50  0001 C CNN
+F 0 "#PWR010" H 10400 2250 50  0001 C CNN
 F 1 "+3.3V" H 10400 2540 50  0000 C CNN
 F 2 "" H 10400 2400 60  0000 C CNN
@@
 REG.
 $Comp
-L GND #PWR018
+L GND #PWR011
 U 1 1 55CFB7D3
 P 10400 1600
-F 0 "#PWR018" H 10400 1350 50  0001 C CNN
+F 0 "#PWR011" H 10400 1350 50  0001 C CNN
 F 1 "GND" H 10400 1450 50  0000 C CNN
 F 2 "" H 10400 1600 60  0000 C CNN
@@
 $EndComp
 $Comp
-L +5V #PWR019
+L +5V #PWR012
 U 1 1 55CFB8E7
 P 10450 1300
-F 0 "#PWR019" H 10450 1150 50  0001 C CNN
+F 0 "#PWR012" H 10450 1150 50  0001 C CNN
 F 1 "+5V" H 10450 1440 50  0000 C CNN
 F 2 "" H 10450 1300 60  0000 C CNN
@@
 DECOUPLING
 $Comp
-L +3.3V #PWR021
+L +3.3V #PWR013
 U 1 1 55CFF1F5
 P 8950 1300
-F 0 "#PWR021" H 8950 1150 50  0001 C CNN
+F 0 "#PWR013" H 8950 1150 50  0001 C CNN
 F 1 "+3.3V" H 8950 1440 50  0000 C CNN
 F 2 "" H 8950 1300 60  0000 C CNN
@@
 A1
 $Comp
-L GND #PWR025
+L GND #PWR014
 U 1 1 55D03D7B
 P 9750 2900
-F 0 "#PWR025" H 9750 2650 50  0001 C CNN
+F 0 "#PWR014" H 9750 2650 50  0001 C CNN
 F 1 "GND" H 9750 2750 50  0000 C CNN
 F 2 "" H 9750 2900 60  0000 C CNN
@@
 Wire Bus Line
 	900  2200 900  800
-Wire Wire Line
-	1000 2300 1500 2300
-Wire Bus Line
-	4200 4200 4200 1700
-Wire Bus Line
-	3800 4200 3800 2500
-Wire Bus Line
-	900  4200 900  2300
+Wire Bus Line
+	4200 1700 4200 4200
+Wire Bus Line
+	3800 2500 3800 4200
+Wire Bus Line
+	900  2300 900  4200
 Wire Wire Line
 	1000 2400 1500 2400
@@
 	1000 2700 1500 2700
 Wire Wire Line
-	3700 2300 3100 2300
-Wire Wire Line
 	3100 2400 3700 2400
 Wire Wire Line
@@
 	7400 1550 7400 2400
 Wire Wire Line
-	7300 2400 7300 1950
+	7300 1950 7300 2400
 Wire Wire Line
 	7200 2050 7300 2050
 Connection ~ 7300 2050
 Wire Wire Line
-	7500 2400 7500 1950
+	7500 1950 7500 2400
 Wire Wire Line
 	7500 2050 7600 2050
@@
 	9750 2900 9750 2750
 Wire Wire Line
-	10400 1600 9250 1600
+	9250 1600 10400 1600
 Wire Wire Line
 	8950 1300 9750 1300
 Wire Bus Line
-	4200 4200 900  4200
+	900  4200 4200 4200
+Text Label 1350 2300 0    39   ~ 0
+A2
+Entry Wire Line
+	3700 2300 3800 2400
 Entry Wire Line
 	900  2200 1000 2300
-Text Label 3650 2300 0    39   ~ 0
-A2
+Wire Wire Line
+	1000 2300 1500 2300
+Wire Wire Line
+	3700 2300 3100 2300
 $EndSCHEMATC
